Commit message: Includes Merged Mesh and Updated irb120.xacro file

File: abby_arm_simu/abby_description/urdf/irb120.xacro (robot description, xacro)
@@ -10,5 +10,5 @@
   #<xacro:property name="camera_link" value="0.05" /> <!-- Size of square 'camera' box -->
   #<xacro:property name="axel_offset" value="0.05" /> <!-- Space btw top of beam and the each joint -->
-  <!-- Import all Gazebo-customization elements, including Gazebo colors -->
+  <!-- Import all Gazebo-customization elements, including Gazebos -->
   <xacro:include filename="$(find abby_description)/urdf/irb120.gazebo" />
   <!-- Import Rviz colors -->
@@ -22,24 +22,7 @@
   <!-- Base Link -->
   <link name="link1">
-    <!--collision>
-      <origin xyz="0 0 0" rpy="0 0 0"/>
-      <geometry>
-	<box size="0.1 0.1 0.1"/>
-      </geometry>
-    </collision-->
-    <!--visual>
-      <origin xyz="0 0 0" rpy="0 0 0"/>
-      <geometry>
-        <mesh filename="package://abb_common/meshes/irb120/visual/base_link.stl"/>
-      </geometry>
-      <material name="abb_orange">
-        <color rgba="1 0.43 0 1"/>
-      </material>
-    </visua-->
-    <visual>
-      <!--origin xyz="0 0 ${height1/2}" rpy="0 0 0"/-->
+    <visual>
        <origin xyz="0 0 0" rpy="0 0 0"/>
       <geometry>
-	<!--box size="${width} ${width} ${height1}"/-->
 	       <mesh filename="package://abb_common/meshes/irb120/visual/base_link.stl"/>
       </geometry>
@@ -65,14 +48,7 @@
   <!-- Middle Link -->
   <link name="link2">
-    <!--collision>
-      <origin xyz="0 0 0" rpy="0 0 0"/>
-      <geometry>
-	<box size="0.1 0.1 0.1"/>
-      </geometry>
-    </collision-->
-    <visual>
-      <origin xyz="0 0 0" rpy="0 0 0"/>
-      <geometry>
-	<!--box size="${width} ${width} ${height2}"/-->
+    <visual>
+      <origin xyz="0 0 0" rpy="0 0 0"/>
+      <geometry>
 	<mesh filename="package://abb_common/meshes/irb120/collision/link_1.stl"/>
       </geometry>
@@ -230,5 +206,5 @@
 	        <mesh filename="package://abb_common/meshes/irb120/visual/link_6.stl"/>
       </geometry>
-      <material name="orange"/>
+      <material name="grey"/>
     </visual>
     <inertial>
@@ -249,4 +225,97 @@
     <dynamics damping="0.7"/>
   </joint>
+  <link name="LBracket">
+    <collision>
+      <origin xyz="0 0 0" rpy="0 0 0"/>
+      <geometry>
+	<box size="0.1 0.1 0.1"/>
+      </geometry>
+    </collision>
+    <visual>
+      <origin xyz="0 0 0" rpy="1.57 0 0"/>
+      <geometry>
+	<mesh filename="package://abb_common/meshes/irb120/visual/LBracket.stl" scale="0.001 0.001 0.001"/>
+      </geometry>
+	<material name="white"/>
+    </visual>
+    <inertial>
+      <origin xyz="0 0 0" rpy="0 0 0"/>
+      <mass value="1"/>
+      <inertia
+	  ixx="1.0" ixy="0.0" ixz="0.0"
+	  iyy="1.0" iyz="0.0"
+	  izz="1.0"/>
+    </inertial>
+  </link>
+  <link name="paint_gun">
+    <collision>
+      <origin xyz="0 0 0" rpy="0 0 0"/>
+      <geometry>
+	<box size="0.1 0.1 0.1"/>
+      </geometry>
+    </collision>
+    <visual>
+      <origin xyz="0.02 -0.025 0.0525" rpy="1.57 1.5 0"/>
+      <geometry>
+	<mesh filename="package://abb_common/meshes/irb120/visual/288048_CAD_model.stl" scale="0.001 0.001 0.001"/>
+      </geometry>
+     <material name="blue"/>
+    </visual>
+    <inertial>
+      <origin xyz="0 0 0" rpy="0 0 0"/>
+      <mass value="1"/>
+      <inertia
+	  ixx="1.0" ixy="0.0" ixz="0.0"
+	  iyy="1.0" iyz="0.0"
+	  izz="1.0"/>
+    </inertial>
+  </link>
+  <link name="paintTriangle">
+    <collision>
+      <origin xyz="0 0 0" rpy="0 0 0"/>
+      <geometry>
+	<box size="0.1 0.1 0.1"/>
+      </geometry>
+    </collision>
+    <visual>
+      <origin xyz="0 0 0" rpy="-3.14 0 0"/>
+      <geometry>
+	<mesh filename="package://abb_common/meshes/irb120/visual/paintTriangle.stl" scale="0.001 0.001 0.001"/>
+      </geometry>
+      <material name="red"/>
+    </visual>
+    <inertial>
+      <origin xyz="0 0 0" rpy="0 0 0"/>
+      <mass value="1"/>
+      <inertia
+	  ixx="1.0" ixy="0.0" ixz="0.0"
+	  iyy="1.0" iyz="0.0"
+	  izz="1.0"/>
+    </inertial>
+  </link>
+  <joint name="firstEffector" type="continuous">
+    <parent link="link7"/>
+    <child link="LBracket"/>
+    <origin rpy="0 1.5 0" xyz="0 0 0"/>
+    <axis xyz="1 0 0"/>
+     <limit effort="20" lower="-6.98132" upper="6.98132" velocity="7.33038"/>
+    <dynamics damping="0.7"/>
+  </joint>
+  <joint name="touchesEnd" type="continuous">
+    <parent link="LBracket"/>
+    <child link="paint_gun"/>
+    <origin rpy="0 0 0" xyz="0 0 -.02"/>
+    <axis xyz="1 0 0"/>
+     <limit effort="20" lower="-6.98132" upper="6.98132" velocity="7.33038"/>
+    <dynamics damping="0.7"/>
+  </joint>
+  <joint name="paintCloud" type="continuous">
+    <parent link="paint_gun"/>
+    <child link="paintTriangle"/>
+    <origin rpy="0 -1.5 3.14" xyz="0 0 0"/>
+    <axis xyz="1 0 0"/>
+     <limit effort="20" lower="-6.98132" upper="6.98132" velocity="7.33038"/>
+    <dynamics damping="0.7"/>
+  </joint>
   <transmission name="tran1">
     <type>transmission_interface/SimpleTransmission</type>

Commit message: Got positioned correctly and removed unnecessary comments

File: abby_arm_simu/abby_description/urdf/irb120.xacro (robot description, xacro)
@@ -248,66 +248,4 @@
     </inertial>
   </link>
- <!-- <link name="paint_gun">
-    <collision>
-      <origin xyz="0 0 0" rpy="0 0 0"/>
-      <geometry>
-	<box size="0.1 0.1 0.1"/>
-      </geometry>
-    </collision>
-    <visual>
-      <origin xyz="0.02 -0.025 0.0525" rpy="1.57 1.5 0"/>
-      <geometry>
-	<mesh filename="package://abb_common/meshes/irb120/visual/288048_CAD_model.stl" scale="0.001 0.001 0.001"/>
-      </geometry>
-     <material name="blue"/>
-    </visual>
-    <inertial>
-      <origin xyz="0 0 0" rpy="0 0 0"/>
-      <mass value="1"/>
-      <inertia
-	  ixx="1.0" ixy="0.0" ixz="0.0"
-	  iyy="1.0" iyz="0.0"
-	  izz="1.0"/>
-    </inertial>
-  </link>
-  <link name="paintTriangle">
-    <collision>
-      <origin xyz="0 0 0" rpy="0 0 0"/>
-      <geometry>
-	<box size="0.1 0.1 0.1"/>
-      </geometry>
-    </collision>
-    <visual>
-      <origin xyz="0 0 0" rpy="-3.14 0 0"/>
-      <geometry>
-	<mesh filename="package://abb_common/meshes/irb120/visual/paintTriangle.stl" scale="0.001 0.001 0.001"/>
-      </geometry>
-      <material name="red"/>
-    </visual>
-    <inertial>
-      <origin xyz="0 0 0" rpy="0 0 0"/>
-      <mass value="1"/>
-      <inertia
-	  ixx="1.0" ixy="0.0" ixz="0.0"
-	  iyy="1.0" iyz="0.0"
-	  izz="1.0"/>
-    </inertial>
-  </link>
-  <joint name="firstEffector" type="continuous">
-    <parent link="link7"/>
-    <child link="LBracket"/>
-    <origin rpy="0 1.5 0" xyz="0 0 0"/>
-    <axis xyz="1 0 0"/>
-     <limit effort="20" lower="-6.98132" upper="6.98132" velocity="7.33038"/>
-    <dynamics damping="0.7"/>
-  </joint>
-  <joint name="touchesEnd" type="continuous">
-    <parent link="LBracket"/>
-    <child link="paint_gun"/>
-    <origin rpy="0 0 0" xyz="0 0 -.02"/>
-    <axis xyz="1 0 0"/>
-     <limit effort="20" lower="-6.98132" upper="6.98132" velocity="7.33038"/>
-    <dynamics damping="0.7"/>
-  </joint> -->
   <joint name="meshMerge" type="continuous">
     <parent link="link7"/>

Commit message: mergedMesh joint updated to fixed joint so now appears in proper place in RVIZ.

File: abby_arm_simu/abby_description/urdf/irb120.xacro (robot description, xacro)
@@ -248,5 +248,5 @@
     </inertial>
   </link>
-  <joint name="meshMerge" type="continuous">
+  <joint name="meshMerge" type="fixed">
     <parent link="link7"/>
     <child link="mergedMesh"/>

Commit message: Repositioning with alternative method for colored parts.  Still not positioned perfectly so continue to work on.

File: abby_arm_simu/abby_description/urdf/irb120.xacro (robot description, xacro)
@@ -225,5 +225,5 @@
     <dynamics damping="0.7"/>
   </joint>
-  <link name="mergedMesh">
+  <link name="LBracket">
     <collision>
       <origin xyz="0 0 0" rpy="0 0 0"/>
@@ -235,5 +235,5 @@
       <origin xyz=".02 0.023 .0015" rpy="-1.57 3.14 1.57"/>
       <geometry>
-	<mesh filename="package://abb_common/meshes/irb120/visual/Merged_Mesh.stl" scale="0.001 0.001 0.001"/>
+	<mesh filename="package://abb_common/meshes/irb120/visual/LBracket.stl" scale="0.001 0.001 0.001"/>
       </geometry>
 	<material name="white"/>
@@ -248,11 +248,61 @@
     </inertial>
   </link>
-  <joint name="meshMerge" type="fixed">
+  <link name="sprayGun">
+    <collision>
+      <origin xyz="0 0 0" rpy="0 0 0"/>
+      <geometry>
+	<box size="0.1 0.1 0.1"/>
+      </geometry>
+    </collision>
+    <visual>
+      <origin xyz="-.05 0.023 .049" rpy="1.57 3 1.57"/>
+      <geometry>
+	<mesh filename="package://abb_common/meshes/irb120/visual/288048_CAD_model.stl" scale="0.001 0.001 0.001"/>
+      </geometry>
+	<material name="grey"/>
+    </visual>
+    <inertial>
+      <origin xyz="0 0 0" rpy="0 0 0"/>
+      <mass value="1"/>
+      <inertia
+	  ixx="1.0" ixy="0.0" ixz="0.0"
+	  iyy="1.0" iyz="0.0"
+	  izz="1.0"/>
+    </inertial>
+  </link>
+  <link name="paintCloud">
+    <visual>
+      <origin xyz=".02 0.023 .0015" rpy="0 0 0"/>
+      <geometry>
+	<mesh filename="package://abb_common/meshes/irb120/visual/paintTriangle.stl" scale="0.001 0.001 0.001"/>
+      </geometry>
+	<material name="red"/>
+    </visual>
+    <inertial>
+      <origin xyz="0 0 0" rpy="0 0 0"/>
+      <mass value="1"/>
+      <inertia
+	  ixx="1.0" ixy="0.0" ixz="0.0"
+	  iyy="1.0" iyz="0.0"
+	  izz="1.0"/>
+    </inertial>
+  </link>
+  <joint name="connectLBracket" type="fixed">
     <parent link="link7"/>
-    <child link="mergedMesh"/>
+    <child link="LBracket"/>
     <origin rpy="0 -1.5 3.14" xyz="0 0 0"/>
     <axis xyz="1 0 0"/>
-     <limit effort="20" lower="-6.98132" upper="6.98132" velocity="7.33038"/>
-    <dynamics damping="0.7"/>
+  </joint>
+  <joint name="mountGun" type="fixed">
+    <parent link="LBracket"/>
+    <child link="sprayGun"/>
+    <origin rpy="0 -1.5 3.14" xyz="0 0 0"/>
+    <axis xyz="1 0 0"/>
+  </joint>
+  <joint name="cloudOfPaint" type="fixed">
+    <parent link="sprayGun"/>
+    <child link="paintCloud"/>
+    <origin rpy="0 -1.5 3.14" xyz="0 0 0"/>
+    <axis xyz="1 0 0"/>
   </joint>
   <transmission name="tran1">

Commit message: about to remove

File: abby_arm_simu/abby_description/urdf/irb120.xacro (robot description, xacro)
@@ -235,5 +235,5 @@
       <origin xyz=".02 0.023 .0015" rpy="-1.57 3.14 1.57"/>
       <geometry>
-	<mesh filename="package://abb_common/meshes/irb120/visual/Merged_Mesh.stl" scale="0.001 0.001 0.001"/>
+	<mesh filename="package://abb_common/meshes/irb120/visual/finalMergedMesh.dae" scale="0.001 0.001 0.001"/>
       </geometry>
 	<material name="white"/>

Commit message: Successfully positioned and colored each new component.

File: abby_arm_simu/abby_description/urdf/irb120.xacro (robot description, xacro)
@@ -255,6 +255,7 @@
       </geometry>
     </collision>
-    <visual>
-      <origin xyz="-.01 0.023 .045" rpy="1.57 3 1.57"/>
+<!--1.79-->
+    <visual>
+      <origin xyz=".021 0.023 .019" rpy="1.65 3.14 1.59"/>
       <geometry>
 	<mesh filename="package://abb_common/meshes/irb120/visual/288048_CAD_model.stl" scale="0.001 0.001 0.001"/>
@@ -273,5 +274,5 @@
   <link name="paintCloud">
     <visual>
-      <origin xyz=".02 0.023 .0015" rpy="0 0 0"/>
+      <origin xyz="-0.005 -.063 0.444" rpy="-1.57 -.1 1.57"/>
       <geometry>
 	<mesh filename="package://abb_common/meshes/irb120/visual/paintTriangle.stl" scale="0.001 0.001 0.001"/>
